File: LEDDCDCBug.kicad_pcb (KiCad board)
At the start: 2 copper layers, 26.5 x 10.2 mm, 18 parts, among them J1 Conn_01x01, J2 Conn_01x01, J3 Conn_01x01, J4 Conn_01x01, J5 Conn_01x01, J6 Conn_01x01, J7 Conn_01x01, J8 Conn_01x01

Commit message: update design calcs based on real component data
Parts:
- renumbered J8 to J6, J6 to J8
Connections:
- net /+V renamed +36V
- net /DATA_EXT renamed /DATA_IN
- net Net-(J7-Pin_1) renamed /DATA_OUT
Changed lines of the file:
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@@
 	(net 0 "")
 	(net 1 "GND")
-	(net 2 "/+V")
-	(net 3 "/DATA_EXT")
+	(net 2 "+36V")
+	(net 3 "/DATA_IN")
 	(net 4 "/BST")
 	(net 5 "/SW")
@@
 	(net 8 "/FB")
 	(net 9 "/RT")
-	(net 10 "Net-(J7-Pin_1)")
+	(net 10 "/DATA_OUT")
 	(footprint "TestPoint:TestPoint_THTPad_D2.5mm_Drill1.2mm"
 		(layer "F.Cu")
@@
 		(descr "THT pad as test Point, diameter 2.5mm, hole diameter 1.2mm ")
 		(tags "test point THT pad")
-		(property "Reference" "J8"
+		(property "Reference" "J6"
 			(at 0 -2.148 0)
 			(layer "F.SilkS")
@@
 			(layers "*.Cu" "*.Mask")
 			(remove_unused_layers no)
-			(net 10 "Net-(J7-Pin_1)")
+			(net 10 "/DATA_OUT")
 			(pinfunction "Pin_1")
 			(pintype "passive")
@@
 			(layers "*.Cu" "*.Mask")
 			(remove_unused_layers no)
-			(net 2 "/+V")
+			(net 2 "+36V")
 			(pinfunction "Pin_1")
 			(pintype "passive")
@@
 			(layers "*.Cu" "*.Mask")
 			(remove_unused_layers no)
-			(net 2 "/+V")
+			(net 2 "+36V")
 			(pinfunction "Pin_1")
 			(pintype "passive")
@@
 			(layers "F.Cu" "F.Paste" "F.Mask")
 			(roundrect_rratio 0.25)
-			(net 2 "/+V")
+			(net 2 "+36V")
 			(pinfunction "VIN")
 			(pintype "input")
@@
 			(layers "F.Cu" "F.Paste" "F.Mask")
 			(roundrect_rratio 0.25)
-			(net 2 "/+V")
+			(net 2 "+36V")
 			(pinfunction "EN")
 			(pintype "input")
@@
 			(layers "*.Cu" "*.Mask")
 			(remove_unused_layers no)
-			(net 3 "/DATA_EXT")
+			(net 3 "/DATA_IN")
 			(pinfunction "Pin_1")
 			(pintype "passive")
@@
 			(layers "*.Cu" "*.Mask")
 			(remove_unused_layers no)
-			(net 10 "Net-(J7-Pin_1)")
+			(net 10 "/DATA_OUT")
 			(pinfunction "Pin_1")
 			(pintype "passive")
@@
 		(layer "F.Cu")
 		(at 156.7 106.4 90)
-		(property "Reference" "J6"
+		(property "Reference" "J8"
 			(at 0 -0.5 90)
 			(unlocked yes)
@@
 			(layers "*.Cu" "*.Mask")
 			(remove_unused_layers no)
-			(net 3 "/DATA_EXT")
+			(net 3 "/DATA_IN")
 			(pinfunction "Pin_2")
 			(pintype "passive")
@@
 			(layers "F.Cu" "F.Paste" "F.Mask")
 			(roundrect_rratio 0.217391)
-			(net 2 "/+V")
+			(net 2 "+36V")
 			(pintype "passive")
 		)
@@
 	(zone
 		(net 2)
-		(net_name "/+V")
+		(net_name "+36V")
 		(layer "F.Cu")
 		(name "40")
